File: hw/i2c485.sch (KiCad schematic (older format))
At the start: 2 parts

Commit message: driver, io, pwr ...
Parts:
- added C? (x4): C, ~, symbol C
- added C? (x2): CP1, ~, symbol CP1
- added D? (x5): ZENER, ~, symbol ZENER
- added D?: DIODE, ~, symbol DIODE
- added IC?: SP3485CN, SO8, symbol SP3485CN
- added P?: CONN_3X2, symbol CONN_3X2
- added R? (x6): R, ~, symbol R
- added U?: 78L05, symbol 78L05
- added X?: CRYSTAL, ~, symbol CRYSTAL
Connections:
- wire segments 10 -> 65

Commit message: netlist
Parts:
- added C1, C2, C3: 100n, ~, symbol C
- added P1, P2: CONN_4, symbol CONN_4
- C10, C9: renamed from C?; value C -> 22p
- C4: renamed from C?; value CP1 -> 100u/35V
- C5, C6, C7: renamed from C?; value C -> 100n
- C8: renamed from C?; value CP1 -> 22u/16V
- D1: renamed from D?; value DIODE -> BAS40
- D2: renamed from D?; value ZENER -> BZX84C 16
- D3, D4, D5, D6: renamed from D?; value ZENER -> BZX84C5V6
- R1, R2: renamed from R?; value R -> 4k7
- R3, R4, R5, R6: renamed from R?; value R -> 10R
- X1: renamed from X?; value CRYSTAL -> 3,6864MHz
- gave numbers to parts that had none: 4
Connections:
- net labels added: 485A, 485B, GNDIN, P1SDA, P2SCL, VIN
- wire segments 65 -> 76
- no-connect marks 0 -> 14
Other:
- moved on the sheet: D3, D4, D5, D6, R3, R4, R5, R6

Commit message: layout - components
Parts:
- added C11: 100n, ~, symbol C
- added R7: 10R, ~, symbol R
- D1: value BAS40 -> 1N4007
- D2: value BZX84C 16 -> SMAJ18A
- D3, D5: value BZX84C5V6 -> SMAJ15CA
- U1: footprint (none) -> ~
Connections:
- net 485A: now also P1.3 (P3); no longer P1.2 (P2)
- net 485B: now also P1.4 (P4); no longer P1.3 (P3)
- net GND: now also C11.2
- net P1SDA: now also P2.3 (P3); no longer P2.2 (P2)
- net P2SCL: now also P2.4 (P4); no longer P2.3 (P3)
- net VCC: now also R7.2; no longer P2.4 (P4)
- net VIN: now also P1.2 (P2); no longer P1.4 (P4)
- new net: C11.1, P2.2 (P2), R7.1
Other:
- moved on the sheet: P1
